File: MCP23S17 Breakout.brd (EAGLE design)
At the start: 30 x 40 mm, 14 parts, among them IC1 MCP23S17SO

Commit message: Update breakout
Parts:
- removed JP7: (no value), pinhead:1X04
- added JP5: (no value), pinhead:1X06
- JP4: device pinhead:1X04 -> pinhead:1X02
- JP6: device pinhead:1X02 -> pinhead:1X06
- moved JP6 30.1 mm to (15.2, 37.4), turned to 0 degrees
- moved JP4 13.4 mm to (26.7, 9.53), turned to 180 degrees
Connections:
- net CS: now also JP5.2, JP6.2; no longer JP4.1, JP7.1
- net GND: now also JP5.1, JP5.6, JP6.1, JP6.6
- net INTA: now also JP4.1; no longer JP6.1
- net INTB: now also JP4.2; no longer JP6.2
- net SCK: now also JP5.3, JP6.3; no longer JP4.2, JP7.2
- net SI: now also JP5.4, JP6.4; no longer JP4.3, JP7.3
- net SO: now also JP5.5, JP6.5; no longer JP4.4, JP7.4
Other:
- board text added: "CC BY-SA 4.0"
- board text added: "Insight, foresight, more sight, The clock on the wall reads a quarter past midnight"
- board text added: "MCP23S17 Breakout v1.0.1"
- board text added: "v1.0.1"
- board text removed: "MCP23S17 Breakout v1.0.0"
- board text removed: "Paul Williamson CC BY-SA 4.0"
- board text removed: "v1.0.0"
Changed lines of the file:
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@@
 <text x="2.54" y="11.43" size="0.8128" layer="21" font="vector" ratio="13" align="bottom-center">GND</text>
 <text x="3.81" y="7.3025" size="0.8128" layer="21" font="vector" ratio="13" rot="R180" align="center">POWER</text>
-<text x="11.43" y="4.445" size="1.27" layer="21" font="vector" ratio="13" rot="R270" align="center-right">CS</text>
-<text x="13.97" y="4.445" size="1.27" layer="21" font="vector" ratio="13" rot="R270" align="center-right">SCK</text>
-<text x="16.51" y="4.445" size="1.27" layer="21" font="vector" ratio="13" rot="R270" align="center-right">SI</text>
+<text x="11.43" y="4.445" size="1.016" layer="21" font="vector" ratio="13" rot="R270" align="center-right">CS</text>
+<text x="13.97" y="4.445" size="1.016" layer="21" font="vector" ratio="13" rot="R270" align="center-right">SCK</text>
+<text x="16.51" y="4.445" size="1.016" layer="21" font="vector" ratio="13" rot="R270" align="center-right">SI</text>
 <text x="8.89" y="32.0675" size="1.016" layer="21" font="vector" ratio="13" align="center-right">1</text>
 <text x="8.89" y="28.8925" size="1.016" layer="21" font="vector" ratio="13" align="center-right">0</text>
@@
 <text x="13.97" y="36.1475" size="1.016" layer="21" font="vector" ratio="13" rot="R90" align="center-right">SCK</text>
 <text x="16.51" y="36.1475" size="1.016" layer="21" font="vector" ratio="13" rot="R90" align="center-right">SI</text>
-<text x="19.05" y="4.445" size="1.27" layer="21" font="vector" ratio="13" rot="R270" align="center-right">SO</text>
+<text x="19.05" y="4.445" size="1.016" layer="21" font="vector" ratio="13" rot="R270" align="center-right">SO</text>
 <text x="19.05" y="36.1475" size="1.016" layer="21" font="vector" ratio="13" rot="R90" align="center-right">SO</text>
 <text x="26.67" y="7.62" size="0.8128" layer="21" font="vector" ratio="13" align="top-center">INTERRUPT</text>
 <text x="27.94" y="11.1125" size="1.27" layer="21" font="vector" ratio="13" rot="R180" align="top-center">A</text>
 <text x="25.4" y="11.1125" size="1.27" layer="21" font="vector" ratio="13" rot="R180" align="top-center">B</text>
-<text x="8.89" y="19.685" size="1.016" layer="22" font="vector" ratio="10" rot="MR90" align="center">https://git.io/v6Mtp</text>
-<text x="13.335" y="20.6375" size="1.016" layer="22" font="vector" ratio="10" rot="MR270" align="center">Paul Williamson
-CC BY-SA 4.0</text>
-<text x="19.3675" y="19.685" size="1.27" layer="22" font="vector" ratio="10" rot="MR270" align="center">MCP23S17 Breakout
-v1.0.0</text>
-<text x="20.32" y="0.635" size="1.016" layer="21" font="vector" ratio="13">v1.0.0</text>
+<text x="13.335" y="19.685" size="1.016" layer="22" font="vector" ratio="10" rot="MR90" align="center">https://git.io/v6Mtp</text>
+<text x="5.3975" y="20.6375" size="1.016" layer="22" font="vector" ratio="10" rot="MR270" align="center">CC BY-SA 4.0</text>
+<text x="19.3675" y="19.685" size="1.4224" layer="22" font="vector" ratio="10" rot="MR270" align="center">MCP23S17 Breakout
+v1.0.1</text>
+<text x="15.24" y="8.255" size="1.016" layer="21" font="vector" ratio="13" align="center">v1.0.1</text>
+<text x="9.525" y="20.32" size="0.8128" layer="22" font="vector" ratio="13" rot="MR270" align="center">Insight, foresight, more sight,
+The clock on the wall
+reads a quarter past midnight</text>
+<text x="8.89" y="4.445" size="1.016" layer="21" font="vector" ratio="13" rot="R270" align="center-right">GND</text>
+<text x="8.89" y="4.445" size="1.016" layer="21" font="vector" ratio="13" rot="R270" align="center-right">GND</text>
+<text x="21.59" y="4.445" size="1.016" layer="21" font="vector" ratio="13" rot="R270" align="center-right">GND</text>
+<text x="21.59" y="4.445" size="1.016" layer="21" font="vector" ratio="13" rot="R270" align="center-right">GND</text>
+<text x="8.89" y="36.195" size="1.016" layer="21" font="vector" ratio="13" rot="R90" align="center-right">GND</text>
+<text x="21.59" y="36.195" size="1.016" layer="21" font="vector" ratio="13" rot="R90" align="center-right">GND</text>
 </plain>
 <attributes>
@@
 <element name="U$3" library="SparkFun-Electromechanical" package="STAND-OFF" value="" x="3" y="3"/>
 <element name="U$4" library="SparkFun-Electromechanical" package="STAND-OFF" value="" x="27" y="3"/>
-<element name="JP6" library="pinhead" package="1X02" value="" x="26.67" y="9.525" smashed="yes" rot="R180">
+<element name="JP4" library="pinhead" package="1X02" value="" x="26.67" y="9.525" smashed="yes" rot="R180">
 <attribute name="VALUE" x="29.21" y="12.7" size="1.27" layer="27" rot="R180"/>
 </element>
-<element name="JP7" library="pinhead" package="1X04" value="" x="15.24" y="37.4175" smashed="yes">
+<element name="JP6" library="pinhead" package="1X06" value="" x="15.24" y="37.4175" smashed="yes">
 <attribute name="VALUE" x="10.16" y="34.2425" size="1.27" layer="27"/>
 </element>
-<element name="JP4" library="pinhead" package="1X04" value="" x="15.24" y="2.54" smashed="yes">
+<element name="JP5" library="pinhead" package="1X06" value="" x="15.24" y="2.54" smashed="yes">
 <attribute name="VALUE" x="10.16" y="-0.635" size="1.27" layer="27"/>
 </element>
@@
 <contactref element="IC1" pad="10"/>
 <contactref element="JP3" pad="2"/>
-<via x="22.86" y="34.29" extent="1-16" drill="0.6"/>
-<via x="22.86" y="5.3975" extent="1-16" drill="0.6"/>
+<via x="24.13" y="34.29" extent="1-16" drill="0.6"/>
+<via x="23.495" y="5.3975" extent="1-16" drill="0.6"/>
 <via x="15.24" y="11.43" extent="1-16" drill="0.6"/>
 <via x="15.24" y="25.4" extent="1-16" drill="0.6"/>
-<via x="7.62" y="34.29" extent="1-16" drill="0.6"/>
+<via x="6.35" y="34.29" extent="1-16" drill="0.6"/>
+<contactref element="JP6" pad="6"/>
+<contactref element="JP6" pad="1"/>
+<contactref element="JP5" pad="6"/>
+<contactref element="JP5" pad="1"/>
+<via x="23.495" y="5.3975" extent="1-16" drill="0.6"/>
+<via x="6.35" y="5.3975" extent="1-16" drill="0.6"/>
 </signal>
 <signal name="SO">
 <contactref element="IC1" pad="14"/>
-<contactref element="JP7" pad="4"/>
-<contactref element="JP4" pad="4"/>
+<contactref element="JP6" pad="5"/>
+<contactref element="JP5" pad="5"/>
 <wire x1="19.05" y1="37.4175" x2="19.05" y2="2.54" width="0.254" layer="16"/>
 <wire x1="10.46" y1="10.16" x2="9.2075" y2="10.16" width="0.254" layer="1"/>
@@
 <signal name="SI">
 <contactref element="IC1" pad="13"/>
-<contactref element="JP7" pad="3"/>
-<contactref element="JP4" pad="3"/>
+<contactref element="JP6" pad="4"/>
+<contactref element="JP5" pad="4"/>
 <wire x1="16.51" y1="37.4175" x2="16.51" y2="2.54" width="0.254" layer="16"/>
 <wire x1="10.46" y1="11.43" x2="9.2075" y2="11.43" width="0.254" layer="1"/>
@@
 <signal name="SCK">
 <contactref element="IC1" pad="12"/>
-<contactref element="JP7" pad="2"/>
-<contactref element="JP4" pad="2"/>
+<contactref element="JP6" pad="3"/>
+<contactref element="JP5" pad="3"/>
 <wire x1="13.97" y1="37.4175" x2="13.97" y2="2.54" width="0.254" layer="16"/>
 <wire x1="10.46" y1="12.7" x2="9.2075" y2="12.7" width="0.254" layer="1"/>
@@
 <signal name="CS">
 <contactref element="IC1" pad="11"/>
-<contactref element="JP7" pad="1"/>
-<contactref element="JP4" pad="1"/>
+<contactref element="JP6" pad="2"/>
+<contactref element="JP5" pad="2"/>
 <wire x1="11.43" y1="37.4175" x2="11.43" y2="2.54" width="0.254" layer="16"/>
 <wire x1="10.46" y1="13.97" x2="9.2075" y2="13.97" width="0.254" layer="1"/>
@@
 <signal name="INTB">
 <contactref element="IC1" pad="19"/>
-<contactref element="JP6" pad="2"/>
+<contactref element="JP4" pad="2"/>
 <wire x1="20.02" y1="15.24" x2="21.59" y2="15.24" width="0.254" layer="1"/>
 <wire x1="21.59" y1="15.24" x2="25.4" y2="11.43" width="0.254" layer="1"/>
@@
 <signal name="INTA">
 <contactref element="IC1" pad="20"/>
-<contactref element="JP6" pad="1"/>
+<contactref element="JP4" pad="1"/>
 <wire x1="20.02" y1="16.51" x2="21.59" y2="16.51" width="0.254" layer="1"/>
 <wire x1="21.59" y1="16.51" x2="27.94" y2="10.16" width="0.254" layer="1"/>
